File: GB-DMG-Headphone-PCB/GB-DMG-Headphone-PCB.sch (KiCad schematic (older format))
At the start: 9 parts, among them J1 Conn_01x04, J2 SJ-3566AN

Commit message: Add files via upload
Other:
- note added: "SPST Switch, Normally Closed\n(grounded enables speaker)\n(headphone insert breaks ground)"
- note removed: "SPDT Switch, Normally Closed\n(grounded enables speaker)\n(headphone insert breaks ground)"
Changed lines of the file:
@@
 	6725 3225 6950 3225
 Text Notes 6975 3425 0    50   ~ 0
-SPDT Switch, Normally Closed\n(grounded enables speaker)\n(headphone insert breaks ground)
+SPST Switch, Normally Closed\n(grounded enables speaker)\n(headphone insert breaks ground)
 Text GLabel 6475 4250 2    50   Input ~ 0
 LEFT
